Commit message: Add moveit package

File: src/SO-ARM100_description/urdf/grippers/gripper_jaw.xacro (robot description, xacro)
@@ -1,18 +1,29 @@
 <robot xmlns:xacro="http://ros.org/wiki/xacro">
-  <link name="gripper">
-    <xacro:default_inertial mass="0.09"/>
-    <visual><geometry><mesh filename="package://so_arm100_description/meshes/Fixed_Jaw.stl"/></geometry><material name="3d_printed"/></visual>
+  <!-- Links -->
+  <xacro:robot_link name="gripper" mesh="Fixed_Jaw" mass="0.0929859" origin="0.00552377 -0.0280167 0.000483583 0 0 0" inertia="5.03136e-05 4.64098e-05 2.72961e-05"/>
+  <link name="moving_jaw">
+    <inertial>
+      <mass value="0.0202444"/>
+      <origin xyz="-0.00161745 -0.0303473 0.000449646" rpy="0 0 0"/>
+      <inertia ixx="1.11265e-05" ixy="0" ixz="0" iyy="8.99651e-06" iyz="0" izz="2.99548e-06"/>
+    </inertial>
+    <visual>
+      <geometry><mesh filename="package://so_arm100_description/meshes/Moving_Jaw.stl"/></geometry>
+      <material name="3d_printed"/>
+    </visual>
+    <collision><geometry><mesh filename="package://so_arm100_description/meshes/Moving_Jaw.stl"/></geometry></collision>
   </link>
-  <link name="jaw">
-    <xacro:default_inertial mass="0.02"/>
-    <visual><geometry><mesh filename="package://so_arm100_description/meshes/Moving_Jaw.stl"/></geometry><material name="3d_printed"/></visual>
-  </link>
-  <joint name="gripper" type="revolute">
-    <parent link="gripper"/>
-    <child link="jaw"/>
-    <origin xyz="-0.0202 -0.0244 0" rpy="0 3.14158 0"/>
-    <axis xyz="0 0 1"/>
-    <limit lower="-0.2" upper="2.0" effort="35" velocity="1"/>
+  <link name="tcp_link"/>
+  <!-- Joints -->
+  <xacro:simple_joint name="gripper" parent="gripper" child="moving_jaw" axis="0 0 1" origin="-0.0202 -0.0244 0 0 3.14158 0" joint_limit="-0.2 2.0"/>
+  <joint name="tool0_to_tcp_link" type="fixed">
+    <parent link="tool0"/>
+    <child link="tcp_link"/>
+    <origin xyz="0 -0.1 0" rpy="0 0 0"/>
   </joint>
-  <xacro:macro name="insert_gripper"/>
+  <!-- Transmissions -->
+  <xacro:if value="${not use_sim_bool}">
+    <xacro:default_transmission motor="jaw"/>
+  </xacro:if>
+  <xacro:macro name="insert_gripper" params="use_sim_bool"/>
 </robot>

File: src/SO-ARM100_description/urdf/grippers/gripper_none.xacro (robot description, xacro)
@@ -3,4 +3,4 @@
     <xacro:default_inertial mass="0.01"/>
   </link>
-  <xacro:macro name="insert_gripper"/>
+  <xacro:macro name="insert_gripper" params="use_sim_bool"/>
 </robot>

File: src/SO-ARM100_description/urdf/so_arm100.urdf.xacro (robot description, xacro)
@@ -10,27 +10,36 @@
   <xacro:include filename="$(find so_arm100_description)/urdf/utils.xacro" />
   <xacro:include filename="$(find so_arm100_description)/urdf/grippers/gripper_$(arg gripper_type).xacro" />
+  <!-- World Link dummy link -->
+  <link name="world"/>
   <!-- Base -->
-  <link name="base">
-    <xacro:default_inertial mass="1.0"/>
-    <visual><geometry><mesh filename="package://so_arm100_description/meshes/Base.stl"/></geometry><material name="3d_printed"/></visual>
-    <visual><geometry><mesh filename="package://so_arm100_description/meshes/Base_Motor.stl"/></geometry><material name="sts3215"/></visual>
-    <collision><geometry><mesh filename="package://so_arm100_description/meshes/Base.stl"/></geometry></collision>
-  </link>
+  <xacro:robot_link name="base" mesh="Base" mass="1.0" origin="0 0 0 0 0 0" inertia="0.01 0.01 0.01"/>
   <!-- Shoulder -->
-  <xacro:robot_link name="shoulder" mesh="Rotation_Pitch" mass="0.119226"/>
+  <xacro:robot_link name="shoulder" mesh="Rotation_Pitch" mass="0.119226" origin="-9.07886e-05 0.0590972 0.031089 0 0 0" inertia="5.94278e-05 5.89975e-05 3.13712e-05"/>
   <!-- Upper arm -->
-  <xacro:robot_link name="upper_arm" mesh="Upper_Arm" mass="0.162409"/>
+  <xacro:robot_link name="upper_arm" mesh="Upper_Arm" mass="0.162409" origin="-1.72052e-05 0.0701802 0.00310545 0 0 0" inertia="0.000213312 0.000167164 7.01522e-05"/>
   <!-- Lower arm -->
-  <xacro:robot_link name="lower_arm" mesh="Lower_Arm" mass="0.147968"/>
+  <xacro:robot_link name="lower_arm" mesh="Lower_Arm" mass="0.147968" origin="-0.00339604 0.00137796 0.0768007 0 0 0" inertia="0.000138803 0.000107748 4.84242e-05"/>
   <!-- Wrist -->
-  <xacro:robot_link name="wrist" mesh="Wrist_Pitch_Roll" mass="0.0661321"/>
+  <xacro:robot_link name="wrist" mesh="Wrist_Pitch_Roll" mass="0.0661321" origin="-0.00852653 -0.0352279 -2.34622e-05 0 0 0" inertia="3.45403e-05 2.39041e-05 1.94704e-05"/>
+  <!-- Tool0 dummy link -->>
+  <link name="tool0"/>
   <!-- Insert the chosen gripper -->
-  <xacro:insert_gripper/>
+  <xacro:insert_gripper use_sim_bool="${use_sim_bool}"/>
   <!-- Joints -->
-  <xacro:simple_joint name="shoulder_pan" parent="base" child="shoulder" axis="0 1 0" origin="0 -0.0452 0.0165 1.57079 0 0"/>
-  <xacro:simple_joint name="shoulder_lift" parent="shoulder" child="upper_arm" axis="1 0 0" origin="0 0.1025 0.0306 -1.8 0 0"/>
-  <xacro:simple_joint name="elbow_flex" parent="upper_arm" child="lower_arm" axis="1 0 0" origin="0 0.11257 0.028 1.57079 0 0"/>
-  <xacro:simple_joint name="wrist_flex" parent="lower_arm" child="wrist" axis="1 0 0" origin="0 0.0052 0.1349 -1 0 0"/>
-  <xacro:simple_joint name="wrist_roll" parent="wrist" child="gripper" axis="0 1 0" origin="0 -0.0601 0 0 1.57079 0"/>
+  <joint name="world_to_base" type="fixed">
+    <parent link="world"/>
+    <child link="base"/>
+    <origin xyz="0 0 0" rpy="0 0 0"/>
+  </joint>
+  <xacro:simple_joint name="shoulder_pan" parent="base" child="shoulder" axis="0 1 0" origin="0 -0.0452 0.0165 1.57079 0 0" joint_limit="-2.0 2.0"/>
+  <xacro:simple_joint name="shoulder_lift" parent="shoulder" child="upper_arm" axis="1 0 0" origin="0 0.1025 0.0306 -1.8 0 0" joint_limit="0 3.5"/>
+  <xacro:simple_joint name="elbow_flex" parent="upper_arm" child="lower_arm" axis="1 0 0" origin="0 0.11257 0.028 1.57079 0 0" joint_limit="-3.14158 0"/>
+  <xacro:simple_joint name="wrist_flex" parent="lower_arm" child="wrist" axis="1 0 0" origin="0 0.0052 0.1349 -1 0 0" joint_limit="-2.5 1.2"/>
+  <xacro:simple_joint name="wrist_roll" parent="wrist" child="tool0" axis="0 1 0" origin="0 -0.0601 0 0 1.57079 0" joint_limit="-3.14158 3.14158"/>
+  <joint name="tool0_to_gripper" type="fixed">
+    <parent link="tool0"/>
+    <child link="gripper"/>
+    <origin xyz="0 0 0" rpy="0 0 0"/>
+  </joint>
   <!-- Transmissions (optional if use_sim == true) -->
   <xacro:if value="${not use_sim_bool}">
@@ -40,5 +49,4 @@
     <xacro:default_transmission motor="4"/>
     <xacro:default_transmission motor="5"/>
-    <xacro:default_transmission motor="6"/>
   </xacro:if>
 </robot>

File: src/SO-ARM100_description/urdf/utils.xacro (robot description, xacro)
@@ -1,13 +1,19 @@
 <robot xmlns:xacro="http://ros.org/wiki/xacro">
-  <xacro:macro name="default_inertial" params="mass">
+  <xacro:macro name="robot_inertial" params="mass origin inertia">
     <inertial>
       <mass value="${mass}"/>
-      <origin xyz="0 0 0" rpy="0 0 0"/>
-      <inertia ixx="0.01" ixy="0" ixz="0" iyy="0.01" iyz="0" izz="0.01"/>
+      <origin xyz="${origin.split()[0]} ${origin.split()[1]} ${origin.split()[2]}"
+              rpy="${origin.split()[3]} ${origin.split()[4]} ${origin.split()[5]}"/>
+      <inertia  ixx="${inertia.split()[0]}"
+                ixy="0"
+                ixz="0"
+                iyy="${inertia.split()[1]}"
+                iyz="0"
+                izz="${inertia.split()[2]}"/>
     </inertial>
   </xacro:macro>
-  <xacro:macro name="robot_link" params="name mesh mass">
+  <xacro:macro name="robot_link" params="name mesh mass origin inertia">
     <link name="${name}">
-      <xacro:default_inertial mass="${mass}"/>
+      <xacro:robot_inertial mass="${mass}" origin="${origin}" inertia="${inertia}"/>
       <visual><geometry><mesh filename="package://so_arm100_description/meshes/${mesh}.stl"/></geometry><material name="3d_printed"/></visual>
       <visual><geometry><mesh filename="package://so_arm100_description/meshes/${mesh}_Motor.stl"/></geometry><material name="sts3215"/></visual>
@@ -15,5 +21,5 @@
     </link>
   </xacro:macro>
-  <xacro:macro name="simple_joint" params="name parent child axis origin">
+  <xacro:macro name="simple_joint" params="name parent child axis origin joint_limit">
     <joint name="${name}" type="revolute">
       <parent link="${parent}"/>
@@ -22,5 +28,5 @@
               rpy="${origin.split()[3]} ${origin.split()[4]} ${origin.split()[5]}"/>
       <axis xyz="${axis}"/>
-      <limit lower="-3.14" upper="3.14" effort="35" velocity="1"/>
+      <limit lower="${joint_limit.split()[0]}" upper="${joint_limit.split()[1]}"  effort="35" velocity="1"/>
     </joint>
   </xacro:macro>
